Commit message: Updated commit with left and right wheels for the robot model

File: my_rb1_description/urdf/my_rb1_robot.urdf (robot description, URDF)
Before this commit: robot rb1, 1 links, 0 joints
Links:
- added link base_footprint
- added link left_wheel, mass 1; collision cylinder length=0.02 radius=0.025; visual cylinder length=0.02 radius=0.025
- added link right_wheel, mass 1; collision cylinder length=0.02 radius=0.025; visual cylinder length=0.02 radius=0.025
Joints:
- added joint base_footprint_joint: type fixed, parent base_link, child base_footprint, origin xyz=0 0 0 rpy=0 0 0
- added joint left_wheel_joint: type continuous, parent base_link, child left_wheel, origin xyz=0  -0.2 -0.15 rpy=0 0 0, axis 0 1 0
- added joint right_wheel_joint: type continuous, parent base_link, child right_wheel, origin xyz=0  0.2 -0.15 rpy=0 0 0, axis 0 1 0

Commit message: Added caster wheel and laser scan

File: my_rb1_description/urdf/my_rb1_robot.urdf (robot description, URDF)
Before this commit: robot rb1, 4 links, 3 joints
Links:
- added link back_caster_wheel, mass 1; collision sphere radius=0.025; visual sphere radius=0.025
- added link front_caster_wheel, mass 1; collision sphere radius=0.025; visual sphere radius=0.025
- added link link_laser, mass 1; collision box size=0.05 0.05 0.1; visual box size=0.05 0.05 0.1
Joints:
- removed joint base_footprint_joint
- added joint back_caster_wheel_joint: type fixed, parent base_link, child back_caster_wheel, origin xyz=0.1  0.0 -0.15 rpy=0 0 0
- added joint front_castor_wheel_joint: type fixed, parent base_link, child front_caster_wheel, origin xyz=-0.1  0.0 -0.15 rpy=0 0 0
- added joint front_laser_joint: type fixed, parent base_link, child link_laser, origin xyz=0.25 0.0 0.075 rpy=3.14159 0 0
- added joint joint_base_link: type fixed, parent base_footprint, child base_link, origin xyz=0.0 0.0 0.15 rpy=0 0 0
- joint left_wheel_joint: limit (none) -> effort=10000 velocity=1000
- joint right_wheel_joint: limit (none) -> effort=10000 velocity=1000

Commit message: Updated launch file

File: my_rb1_description/urdf/my_rb1_robot.urdf (robot description, URDF)
Before this commit: robot rb1, 7 links, 6 joints
Links:
- removed link link_laser
- added link front_laser, mass 1; collision box size=0.05 0.05 0.1; visual box size=0.05 0.05 0.1
Joints:
- removed joint left_wheel_joint
- removed joint right_wheel_joint
- added joint joint_chassis_right_wheel: type continuous, parent base_link, child right_wheel, origin xyz=0  0.2 -0.15 rpy=0 0 0, axis 0 1 0, limit effort=10000 velocity=1000
- added joint joint_left_wheel: type continuous, parent base_link, child left_wheel, origin xyz=0  -0.2 -0.15 rpy=0 0 0, axis 0 1 0, limit effort=10000 velocity=1000

Commit message: Added gazebo tags and it's launch file for simulation

File: my_rb1_description/urdf/my_rb1_robot.urdf (robot description, URDF)
Before this commit: robot robot, 7 links, 6 joints
Links:
- link front_laser: geometry collision box size=0.05 0.05 0.05; visual box size=0.05 0.05 0.05
Joints:
- joint front_laser_joint: child link_laser -> front_laser

Commit message: Updating gazebo launch file

File: my_rb1_description/urdf/my_rb1_robot.urdf (robot description, URDF)
Before this commit: robot robot, 7 links, 6 joints
Joints:
- removed joint front_castor_wheel_joint
- removed joint joint_left_wheel
- added joint front_caster_wheel_joint: type fixed, parent base_link, child front_caster_wheel, origin xyz=-0.1  0.0 -0.15 rpy=0 0 0
- added joint joint_chassis_left_wheel: type continuous, parent base_link, child left_wheel, origin xyz=0  -0.2 -0.15 rpy=0 0 0, axis 0 1 0, limit effort=10000 velocity=1000

Commit message: Update my_rb1_robot.urdf

File: my_rb1_description/urdf/my_rb1_robot.urdf (robot description, URDF)
Before this commit: robot robot, 7 links, 6 joints
Joints:
- joint back_caster_wheel_joint: origin xyz=0.1  0.0 -0.15 rpy=0 0 0 -> xyz=-0.1  0.0 -0.15 rpy=0 0 0
- joint front_caster_wheel_joint: origin xyz=-0.1  0.0 -0.15 rpy=0 0 0 -> xyz=0.1  0.0 -0.15 rpy=0 0 0
- joint joint_chassis_left_wheel: origin xyz=0  -0.2 -0.15 rpy=0 0 0 -> xyz=0  0.2 -0.15 rpy=0 0 0
- joint joint_chassis_right_wheel: origin xyz=0  0.2 -0.15 rpy=0 0 0 -> xyz=0  -0.2 -0.15 rpy=0 0 0

Commit message: Update my_rb1_robot.urdf
Corrected friction and inertial parameters of the wheel to get a proper simulation of the robot.

File: my_rb1_description/urdf/my_rb1_robot.urdf (robot description, URDF)
Before this commit: robot robot, 7 links, 6 joints
Joints:
- joint back_caster_wheel_joint: origin xyz=-0.1  0.0 -0.15 rpy=0 0 0 -> xyz=0.1  0.0 -0.15 rpy=0 0 0

Commit message: Update on caster wheel of the robot

File: my_rb1_description/urdf/my_rb1_robot.urdf (robot description, URDF)
Before this commit: robot robot, 7 links, 6 joints
Joints:
- joint back_caster_wheel_joint: origin xyz=0.1  0.0 -0.15 rpy=0 0 0 -> xyz=-0.1  0.0 -0.15 rpy=0 0 0
